File: hardware/sparkpunk_sequencer.sch (EAGLE design)
At the start: 139 parts, among them IC1 7555, IC3 LM358, IC4 LM358, IC5 CD4013B, IC6 CD4017, Q100 2N3904, Q1000 2N3904, Q200 2N3904, Q300 2N3904, Q400 2N3904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

Commit message: PCB updates after review
Parts:
- removed R12, R9: 10k, SparkFun-Resistors:RESISTOREZ
- added JP3: TEMPO_CV, SparkFun-Connectors:M01SMDNS
- added LOGO4: SFE_LOGO_NAME_FLAME.4_INCH, SparkFun-Aesthetics:SFE_LOGO_NAME_FLAME.4_INCH
- added R20, R21, R22, R25: 10k, SparkFun-Resistors:RESISTOREZ
- added R23, R24: 10k*, SparkFun-Resistors:RESISTOREZ
- added SJ6**: NON-INV-N.O., SparkFun-Passives:SOLDERJUMPERPTH
- JP10: value TRANSPOSE -> TNG-GND
- R10: value 10k -> 10k*
- S3: value SWITCH-MOMENTARY-LEDEZ -> Play Button
- SJ1: value RUN -> RUN-N.C.
- SJ2: value STOP -> STOP-N.C.
- SJ3: value CLK -> CLK-N.C.
- SJ4: value BTN -> BTN-N.C.
- SJ5: value ONE-SHOT -> ONE-SHOT-N.O.
Connections:
- removed net CVSUM: IC3G$1.+IN, R10.1, R12.1
- new net N$64: IC3G2.-IN, R20.1, R25.2
- new net N$65: IC3G2.+IN, R21.2, R22.2
- new net VREF: IC3G1.+IN, R23.1, R24.2, SJ6**.2
- net GND: now also IC3G1.V-, IC4G1.V-, R24.1, R25.1; no longer IC3G$1.V-, IC4G$1.V-, R9.1
- net N$11: now also IC4G1.+IN; no longer IC4G$1.+IN
- net N$12: now also R7.1; no longer R7.2
- net N$15: now also IC3G1.-IN, R10.1; no longer IC3G$1.-IN, R9.2
- net N$16: now also R22.1; no longer R12.2
- net N$17: now also R20.2; no longer IC3G$2.-IN
- net N$18: now also R21.1; no longer IC3G$2.+IN
- net N$19: now also IC3G2.OUT; no longer IC3G$2.OUT
- net N$20: now also IC4G1.-IN, IC4G1.OUT, IC4G2.+IN; no longer IC4G$1.-IN, IC4G$1.OUT, IC4G$2.+IN
- net N$22: now also IC4G2.-IN; no longer IC4G$2.-IN
- net N$23: now also IC4G2.OUT; no longer IC4G$2.OUT
- net N$6: now also IC3G1.OUT; no longer IC3G$1.OUT
- net N$7: now also JP3.1
- net POTSUM: now also SJ6**.1
- net VCC: now also IC3G1.V+, IC4G1.V+, R23.2, R7.2; no longer IC3G$1.V+, IC4G$1.V+, R7.1
Other:
- note added: "* = For inverting summing (higher slider position means lower voltage out, to drive SparkPunk, or other 555-based device), populate R10, R23, R24."
- note added: "** = For non-inverting summing (higher slider yields higher voltage to drive regular VCOs), omit R10, R23, R24, and bridge SJ6."
- note added: "At each rising edge of clock, selects the next step. Reset when last step is active, and held in reset when not running."
- note added: "Divides 7555 output by 2, resulting in 50% duty cycle waveform."
- note added: "Each time S3 is pressed, the output of IC5A toggles."
- note added: "Generates step advance clock. Only active when in running mode."
- note added: "IC3G1 sums the diode or'ed voltages from the step sliders, and optionally invert them. RV2 and C3 form an adjustable lowpass on the resulting voltage. IC3G2 buffers the lowpass, and adds in the external voltage applied to the transpose input"
- note added: "IC4G1 sums the gate voltage from the active step with the 50% duty clock. IC4G2 is a comparator with it's trip voltage set by the S5. In legato setting, gate signal will be active for whole step when step switch is on. On non-legato, gate will be active for 1/2 of a step when the switch is on."
- note added: "One step is selected at a time by the CD4017. This turns on the transistor, lighting the step LED. The slide pot and switch place the voltage on the POTSUM and GATESUM busses, respectively, each combined using a diode-or circuit."
- note added: "S5 selects trip voltage Open = VCC x .8 Closeed = VCC x .32"
- moved on the sheet: BAT1, C3, JP1, JP10, JP2, JP7, R10, R11, R13, R15, R16, R17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

Commit message: Small updates after creating BOM
Parts:
- C1: value .1 -> .1uf
Other:
- moved on the sheet: R4
Changed lines of the file:
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@@
 </part>
 <part name="SUPPLY6" library="SparkFun-Aesthetics" deviceset="VCC" device=""/>
-<part name="C1" library="SparkFun-Capacitors" deviceset="0.1UF-50V-20%(PTH)" device="KIT-EZ" value=".1"/>
+<part name="C1" library="SparkFun-Capacitors" deviceset="0.1UF-50V-20%(PTH)" device="KIT-EZ" value=".1uf"/>
 <part name="R6" library="SparkFun-Resistors" deviceset="RESISTOR" device="EZ" value="2.2k">
 <attribute name="PROD_ID" value="RES-10691"/>
@@
 <attribute name="PROD_ID" x="50.8" y="228.6" size="1.778" layer="96" rot="R90" display="off"/>
 </instance>
-<instance part="R4" gate="G$1" x="22.86" y="226.06" rot="R90">
-<attribute name="PROD_ID" x="22.86" y="226.06" size="1.778" layer="96" rot="R90" display="off"/>
+<instance part="R4" gate="G$1" x="25.4" y="226.06" rot="R90">
+<attribute name="PROD_ID" x="25.4" y="226.06" size="1.778" layer="96" rot="R90" display="off"/>
 </instance>
 <instance part="SUPPLY6" gate="1" x="35.56" y="261.62"/>
@@
 <pinref part="R4" gate="G$1" pin="1"/>
 <wire x1="43.18" y1="218.44" x2="43.18" y2="215.9" width="0.1524" layer="91"/>
-<wire x1="22.86" y1="220.98" x2="22.86" y2="218.44" width="0.1524" layer="91"/>
-<wire x1="22.86" y1="218.44" x2="43.18" y2="218.44" width="0.1524" layer="91"/>
+<wire x1="25.4" y1="220.98" x2="25.4" y2="218.44" width="0.1524" layer="91"/>
+<wire x1="25.4" y1="218.44" x2="43.18" y2="218.44" width="0.1524" layer="91"/>
 <junction x="43.18" y="218.44"/>
 <pinref part="C1" gate="G$1" pin="2"/>
-<wire x1="22.86" y1="218.44" x2="15.24" y2="218.44" width="0.1524" layer="91"/>
+<wire x1="25.4" y1="218.44" x2="15.24" y2="218.44" width="0.1524" layer="91"/>
 <wire x1="15.24" y1="218.44" x2="15.24" y2="220.98" width="0.1524" layer="91"/>
-<junction x="22.86" y="218.44"/>
+<junction x="25.4" y="218.44"/>
 <pinref part="R6" gate="G$1" pin="1"/>
 <wire x1="7.62" y1="220.98" x2="7.62" y2="218.44" width="0.1524" layer="91"/>
@@
 <segment>
 <pinref part="R4" gate="G$1" pin="2"/>
-<wire x1="15.24" y1="233.68" x2="22.86" y2="233.68" width="0.1524" layer="91"/>
-<wire x1="22.86" y1="233.68" x2="22.86" y2="231.14" width="0.1524" layer="91"/>
+<wire x1="15.24" y1="233.68" x2="25.4" y2="233.68" width="0.1524" layer="91"/>
+<wire x1="25.4" y1="233.68" x2="25.4" y2="231.14" width="0.1524" layer="91"/>
 <pinref part="C1" gate="G$1" pin="1"/>
 <wire x1="15.24" y1="228.6" x2="15.24" y2="233.68" width="0.1524" layer="91"/>
@@
 <wire x1="15.24" y1="256.54" x2="20.32" y2="256.54" width="0.1524" layer="91"/>
 <wire x1="15.24" y1="256.54" x2="15.24" y2="233.68" width="0.1524" layer="91"/>
-<wire x1="22.86" y1="233.68" x2="22.86" y2="243.84" width="0.1524" layer="91"/>
+<wire x1="25.4" y1="233.68" x2="25.4" y2="243.84" width="0.1524" layer="91"/>
 <pinref part="SJ4" gate="1" pin="1"/>
-<wire x1="22.86" y1="243.84" x2="30.48" y2="243.84" width="0.1524" layer="91"/>
-<junction x="22.86" y="233.68"/>
-</segment>
-</net>
+<wire x1="25.4" y1="243.84" x2="30.48" y2="243.84" width="0.1524" layer="91"/>
+<junction x="25.4" y="233.68"/>
+</segment>
+</net>

Commit message: Ready for second prototype
Many changes based on prototype evaluation.
Parts:
- removed JP10: TNG-GND, SparkFun-Connectors:M01SMDNS
- removed R11: 47, SparkFun-Resistors:RESISTOREZ
- removed R8: 10k, SparkFun-Resistors:RESISTOREZ
- removed SJ6**: NON-INV-N.O., SparkFun-Passives:SOLDERJUMPERPTH
- added C10: 1nf, SparkFun-Capacitors:CAPKIT
- added D3: 1N5819, SparkFun-DiscreteSemi:DIODE
- added IC2: LM358, SparkFun-AnalogIC:LM358KIT
- added JP4: CV2, SparkFun-Connectors:M01SMDNS
- added JP5: CV, SparkFun-Connectors:M01SMDNS
- added JP6: VCC, SparkFun-Connectors:M01SMDNS
- added R12: 10k, SparkFun-Resistors:RESISTOREZ
- added R26, R9: 1k, SparkFun-Resistors:RESISTOREZ
- added R27, R28: 100k, SparkFun-Resistors:RESISTOREZ
- added R29: 33k, SparkFun-Resistors:RESISTOREZ
- added R30: 22k, SparkFun-Resistors:RESISTOREZ
- added S1: SPDT, SparkFun-Electromechanical:SWITCH-SPDTKIT
- BAT1: device SparkFun-Connectors:BC9VPC -> SparkFun-Connectors:BC9VPCKIT_SOLDERMASK
- JP2: value CV -> CV1
- JP7: value TRANSPOSE -> GND
- R10: value 10k* -> 1k
- R17: value 47k -> 22k; PROD_ID RES-10687 -> RES-10688
- R18: value 330k -> 22k; PROD_ID RES-10685 -> RES-10688
- R20, R5: value 10k -> 47k; PROD_ID RES-09435 -> RES-10687
- R22: value 10k -> 1k
- R23, R24: value 10k* -> 10k
Connections:
- removed net N$12: IC1.DIS, R7.1
- removed net N$20 (its old number): IC4G1.-IN, IC4G1.OUT, IC4G2.+IN
- removed net VREF: IC3G1.+IN, R23.1, R24.2, SJ6**.2
- new net 555OUT: IC1.OUT, R1.1
- new net N$66: IC2G1.OUT, R10.1, R26.1, R27.1
- new net N$67: JP4.1, R26.2
- new net N$68: JP2.1, R10.2
- new net N$69: IC2G2.-IN, IC4G2.OUT, R21.2
- new net N$70: IC4G2.+IN, R23.2, R24.1
- new net N$71: D3.A, S1.P
- new net VBATT: BAT1.V+, S1.O
- net CLK-IN: now also LED1.A, R13.1
- net CLK-OUT: no longer LED1.A, R13.1
- net GATESUM: now also IC4G1.+IN, R25.2; no longer R5.1
- net GND: now also C10.2, IC2G1.V-, JP7.1, R12.2, R17.1, R23.1, R29.1, R5.1; no longer JP10.1, R18.1, R24.1, S5.O
- net N$11: now also IC4G1.-IN, IC4G1.OUT, R18.2; no longer IC4G1.+IN, R13.2, R5.2
- net N$14: now also C10.1
- net N$15: now also IC3G1.+IN, R12.1, R9.2; no longer IC3G1.-IN, R10.1, R8.1
- net N$16: now also R22.2, R9.1; no longer JP7.1, R22.1
- net N$17: now also IC2G1.-IN, R27.2, R28.1; no longer JP2.1, R11.2, R20.2
- net N$18: now also IC3G2.+IN; no longer R21.1
- net N$19: now also IC2G1.+IN, R20.1, R29.2; no longer IC3G2.OUT, R11.1
- net N$22: now also IC2G2.+IN, R5.2, S5.P; no longer IC4G2.-IN, R17.2
- net N$23: now also IC2G2.OUT; no longer IC4G2.OUT
- net N$25: now also R17.2, S5.O; no longer R17.1, R18.2, S5.P
- net N$6: now also IC3G1.-IN; no longer R8.2
- net N$64: now also IC4G2.-IN, R13.2, R18.1, R21.1, R30.1; no longer IC3G2.-IN, R20.1, R25.2
- net N$65: now also IC3G2.-IN, IC3G2.OUT, JP5.1, R28.2; no longer IC3G2.+IN, R21.2, R22.2
- net POTSUM: now also R22.1; no longer R10.2, SJ6**.1
- net PRECLK: now also IC1.DIS, R7.1; no longer IC1.OUT, R1.1
- net RUN-IN: now also R30.2, S3.A
- net RUN-OUT: no longer S3.A
- net VCC: now also D3.C, IC2G1.V+, JP6.1, R20.2, R24.2; no longer BAT1.V+, R23.2
Other:
- note added: "Approx 3.7 VDC"
- note added: "IC3G1 scales and buffers the voltage from the slider wipers - scaled to a range that doesn't clip the opamp by getting too close to the 9V rail. RV2 and C3 form an adjustable lowpass on the resulting voltage, buffered by IC3G2. IC2G1 inverts, shifts and scales that to a range suitable to drive 555's. A 555's CV range is centered between the rails, and has an inverse voltage-to-frequency response."
- note added: "IC4G1 buffers the gate switch output. IC4G2 adds scaled versions of the 50% step clock and running signal. The result is a stair-step waveform of clock superimposed on gate. IC2G2 is a comparator that trips when the stair-step waveform crosses a threshold. The threshold can be set for long or short steps. See the SPICE sims for more detailed waveforms."
- note added: "ON/OFF"
- note added: "S5 selects trip voltage Open = VCC x .8 Closed = VCC x .32"
- note added: "V02"
- note removed: "* = For inverting summing (higher slider position means lower voltage out, to drive SparkPunk, or other 555-based device), populate R10, R23, R24."
- note removed: "** = For non-inverting summing (higher slider yields higher voltage to drive regular VCOs), omit R10, R23, R24, and bridge SJ6."
- note removed: "Ground transpose input if unused."
- note removed: "IC3G1 sums the diode or'ed voltages from the step sliders, and optionally invert them. RV2 and C3 form an adjustable lowpass on the resulting voltage. IC3G2 buffers the lowpass, and adds in the external voltage applied to the transpose input"
- note removed: "IC4G1 sums the gate voltage from the active step with the 50% duty clock. IC4G2 is a comparator with it's trip voltage set by the S5. In legato setting, gate signal will be active for whole step when step switch is on. On non-legato, gate will be active for 1/2 of a step when the switch is on."
- note removed: "S5 selects trip voltage Open = VCC x .8 Closeed = VCC x .32"
- note removed: "V01"
- moved on the sheet: BAT1, C3, C5, C6, C9, D1, D2, IC3G1, IC3G2, IC4G1, IC4G2, IC5P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

Commit message: After library updates
Picking up PROD_ID's for a few parts that didn't have them before.

No changes to the layout.
Parts:
- IC5: PROD_ID (none) -> IC-11930
- R10, R22, R26, R9: PROD_ID RES-09435 -> RES-08380
Changed lines of the file:
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@@
 <part name="JP2" library="SparkFun-Connectors" deviceset="M01" device="SMDNS" value="CV1"/>
 <part name="IC4" library="SparkFun-AnalogIC" deviceset="LM358" device="KIT" value="LM358"/>
-<part name="IC5" library="SparkFun-DigitalIC" deviceset="CD4013" device="" value="CD4013B"/>
+<part name="IC5" library="SparkFun-DigitalIC" deviceset="CD4013" device="" value="CD4013B">
+<attribute name="PROD_ID" value="IC-11930"/>
+</part>
 <part name="D100" library="SparkFun-DiscreteSemi" deviceset="DIODE" device="" value="1N5819">
 <attribute name="PROD_ID" value="DIO-11895"/>
@@
 </part>
 <part name="R22" library="SparkFun-Resistors" deviceset="RESISTOR" device="EZ" value="1k">
-<attribute name="PROD_ID" value="RES-09435"/>
+<attribute name="PROD_ID" value="RES-08380"/>
 </part>
 <part name="R9" library="SparkFun-Resistors" deviceset="RESISTOR" device="EZ" value="1k">
-<attribute name="PROD_ID" value="RES-09435"/>
+<attribute name="PROD_ID" value="RES-08380"/>
 </part>
 <part name="JP4" library="SparkFun-Connectors" deviceset="M01" device="SMDNS" value="CV2"/>
@@
 <part name="IC2" library="SparkFun-AnalogIC" deviceset="LM358" device="KIT" value="LM358"/>
 <part name="R10" library="SparkFun-Resistors" deviceset="RESISTOR" device="EZ" value="1k">
-<attribute name="PROD_ID" value="RES-09435"/>
+<attribute name="PROD_ID" value="RES-08380"/>
 </part>
 <part name="R26" library="SparkFun-Resistors" deviceset="RESISTOR" device="EZ" value="1k">
-<attribute name="PROD_ID" value="RES-09435"/>
+<attribute name="PROD_ID" value="RES-08380"/>
 </part>
 <part name="R27" library="SparkFun-Resistors" deviceset="RESISTOR" device="EZ" value="100k">

Commit message: Ready for red review
Incorporating all changes from second round of protos, builder feedback,
etc.
Parts:
- added C11: .1uf, SparkFun-Capacitors:0.1UF-50V-20%(PTH)KIT-EZ
- C9: value 10uf -> 1000uf/25V; device SparkFun-Capacitors:10UF-25V-20%(PTH)KIT -> SparkFun-Capacitors:1000UF-25V(PTH)KIT
Connections:
- net N$63: now also C11.2
- net VCC: now also C11.1
Other:
- note added: "V10"
- note removed: "V02"
- moved on the sheet: C1, C9, R14, R2, R6, S3, SJ4, SJ5

Commit message: Updating for release
Mainly bringing SPICE files to match final implementation, small
notation change on Eagle schematic
Other:
- note added: "S5 selects trip voltage Open = VCC x .32 Closed = VCC x .13"
- note removed: "S5 selects trip voltage Open = VCC x .8 Closed = VCC x .32"
Changed lines of the file:
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@@
 <text x="78.74" y="5.08" size="1.778" layer="97" font="vector">Place near IC1</text>
 <wire x1="101.6" y1="279.4" x2="101.6" y2="210.82" width="0.1524" layer="97" style="shortdash"/>
-<text x="55.88" y="34.036" size="2.54" layer="97" font="vector">Power and decoupling</text>
+<text x="55.88" y="39.116" size="2.54" layer="97" font="vector">Power and decoupling</text>
 <wire x1="101.6" y1="210.82" x2="101.6" y2="149.86" width="0.1524" layer="97" style="shortdash"/>
 <wire x1="101.6" y1="149.86" x2="101.6" y2="106.68" width="0.1524" layer="97" style="shortdash"/>
@@
 See the SPICE sims for more detailed waveforms.</text>
 <text x="391.16" y="53.34" size="1.778" layer="97" font="vector">S5 selects trip voltage
-Open = VCC x .8
-Closed = VCC x .32</text>
+Open = VCC x .32
+Closed = VCC x .13</text>
 <text x="213.36" y="187.96" size="1.778" layer="97" font="vector">One step is selected at a time by the CD4017.
 This turns on the transistor, lighting the step LED.
